File: nova1200rev3pcb/frontpanel.kicad_pcb (KiCad board)
At the start: 2 copper layers, 449.6 x 130.6 mm, 67 parts

Commit message: Added mounting holes (total to 6) to attach front to frontpanel PCB
Also drawn the line through AC0--AC3 pointing to examine and deposit text
Parts:
- added PAD1: MountingHole_Pad, MountingHole:MountingHole_3.2mm_M3, F.Cu at (242.3, 19.1)
- added PAD1: MountingHole_Pad, MountingHole:MountingHole_3.2mm_M3, F.Cu at (242.3, 113.0)
- added PAD1: MountingHole_Pad, MountingHole:MountingHole_3.2mm_M3, F.Cu at (43.2, 113.0)
- added PAD1: MountingHole_Pad, MountingHole:MountingHole_3.2mm_M3, F.Cu at (43.2, 19.1)
- PAD5, PAD6: footprint MountingHole:MountingHole_3.2mm_M3_Pad -> MountingHole:MountingHole_3.2mm_M3
Changed lines of the file:
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@@
     (tracks 0)
     (zones 0)
-    (modules 67)
+    (modules 71)
     (nets 2)
   )
@@
   (layers
     (0 F.Cu signal)
-    (31 B.Cu signal hide)
-    (37 F.SilkS user hide)
-    (38 B.Mask user hide)
-    (39 F.Mask user hide)
-    (40 Dwgs.User user hide)
-    (41 Cmts.User user hide)
+    (31 B.Cu signal)
+    (37 F.SilkS user)
+    (38 B.Mask user)
+    (39 F.Mask user)
+    (40 Dwgs.User user)
+    (41 Cmts.User user)
     (42 Eco1.User user hide)
-    (43 Eco2.User user hide)
+    (43 Eco2.User user)
     (44 Edge.Cuts user)
-    (45 Margin user hide)
-    (46 B.CrtYd user hide)
-    (47 F.CrtYd user hide)
+    (45 Margin user)
+    (46 B.CrtYd user)
+    (47 F.CrtYd user)
   )
   (setup
@@
     (add_net /GND)
   )
-  (module MountingHole:MountingHole_3.2mm_M3_Pad (layer F.Cu)
+  (module MountingHole:MountingHole_3.2mm_M3 (layer F.Cu)
+    (at 242.316 19.05)
+    (descr "Mounting Hole 3.2mm, no annular, M3")
+    (tags "mounting hole 3.2mm no annular m3")
+    (attr virtual)
+    (fp_text reference PAD1 (at 0 0.254) (layer F.SilkS)
+      (effects (font (size 1 1) (thickness 0.15)))
+    )
+    (fp_text value MountingHole_Pad (at 0 4.2) (layer F.Fab)
+      (effects (font (size 1 1) (thickness 0.15)))
+    )
+    (fp_circle (center 0 0) (end 3.45 0) (layer F.CrtYd) (width 0.05))
+    (fp_circle (center 0 0) (end 3.2 0) (layer Cmts.User) (width 0.15))
+    (fp_text user %R (at 0.3 0) (layer F.Fab)
+      (effects (font (size 1 1) (thickness 0.15)))
+    )
+    (pad 1 np_thru_hole circle (at 0 0) (size 3.2 3.2) (drill 3.2) (layers *.Cu *.Mask))
+  )
+  (module MountingHole:MountingHole_3.2mm_M3 (layer F.Cu)
+    (at 242.316 113.03)
+    (descr "Mounting Hole 3.2mm, no annular, M3")
+    (tags "mounting hole 3.2mm no annular m3")
+    (attr virtual)
+    (fp_text reference PAD1 (at 0 0) (layer F.SilkS)
+      (effects (font (size 1 1) (thickness 0.15)))
+    )
+    (fp_text value MountingHole_Pad (at 0 4.2) (layer F.Fab)
+      (effects (font (size 1 1) (thickness 0.15)))
+    )
+    (fp_circle (center 0 0) (end 3.45 0) (layer F.CrtYd) (width 0.05))
+    (fp_circle (center 0 0) (end 3.2 0) (layer Cmts.User) (width 0.15))
+    (fp_text user %R (at 0.3 0) (layer F.Fab)
+      (effects (font (size 1 1) (thickness 0.15)))
+    )
+    (pad 1 np_thru_hole circle (at 0 0) (size 3.2 3.2) (drill 3.2) (layers *.Cu *.Mask))
+  )
+  (module MountingHole:MountingHole_3.2mm_M3 (layer F.Cu)
+    (at 43.18 113.03)
+    (descr "Mounting Hole 3.2mm, no annular, M3")
+    (tags "mounting hole 3.2mm no annular m3")
+    (attr virtual)
+    (fp_text reference PAD1 (at 0 0) (layer F.SilkS)
+      (effects (font (size 1 1) (thickness 0.15)))
+    )
+    (fp_text value MountingHole_Pad (at 0 4.2) (layer F.Fab)
+      (effects (font (size 1 1) (thickness 0.15)))
+    )
+    (fp_circle (center 0 0) (end 3.45 0) (layer F.CrtYd) (width 0.05))
+    (fp_circle (center 0 0) (end 3.2 0) (layer Cmts.User) (width 0.15))
+    (fp_text user %R (at 0.3 0) (layer F.Fab)
+      (effects (font (size 1 1) (thickness 0.15)))
+    )
+    (pad 1 np_thru_hole circle (at 0 0) (size 3.2 3.2) (drill 3.2) (layers *.Cu *.Mask))
+  )
+  (module MountingHole:MountingHole_3.2mm_M3 (layer F.Cu)
+    (at 43.18 19.05)
+    (descr "Mounting Hole 3.2mm, no annular, M3")
+    (tags "mounting hole 3.2mm no annular m3")
+    (attr virtual)
+    (fp_text reference PAD1 (at 0 0) (layer F.SilkS)
+      (effects (font (size 1 1) (thickness 0.15)))
+    )
+    (fp_text value MountingHole_Pad (at 0 4.2) (layer F.Fab)
+      (effects (font (size 1 1) (thickness 0.15)))
+    )
+    (fp_circle (center 0 0) (end 3.45 0) (layer F.CrtYd) (width 0.05))
+    (fp_circle (center 0 0) (end 3.2 0) (layer Cmts.User) (width 0.15))
+    (fp_text user %R (at 0.3 0) (layer F.Fab)
+      (effects (font (size 1 1) (thickness 0.15)))
+    )
+    (pad 1 np_thru_hole circle (at 0 0) (size 3.2 3.2) (drill 3.2) (layers *.Cu *.Mask))
+  )
+  (module MountingHole:MountingHole_3.2mm_M3 (layer F.Cu)
     (at 415.29 19.05)
-    (descr "Mounting Hole 3.2mm, M3")
-    (tags "mounting hole 3.2mm m3")
+    (descr "Mounting Hole 3.2mm, no annular, M3")
+    (tags "mounting hole 3.2mm no annular m3")
     (attr virtual)
-    (fp_text reference PAD6 (at 0 0.254) (layer F.SilkS)
+    (fp_text reference PAD6 (at -0.254 -0.254) (layer F.SilkS)
       (effects (font (size 1 1) (thickness 0.15)))
     )
@@
       (effects (font (size 1 1) (thickness 0.15)))
     )
-    (pad 1 thru_hole circle (at 0 0) (size 6.4 6.4) (drill 3.2) (layers *.Cu *.Mask)
+    (pad 1 np_thru_hole circle (at 0 0) (size 3.2 3.2) (drill 3.2) (layers *.Cu *.Mask)
       (net 1 /GND))
   )
-  (module MountingHole:MountingHole_3.2mm_M3_Pad (layer F.Cu)
+  (module MountingHole:MountingHole_3.2mm_M3 (layer F.Cu)
     (at 415.29 113.03)
-    (descr "Mounting Hole 3.2mm, M3")
-    (tags "mounting hole 3.2mm m3")
+    (descr "Mounting Hole 3.2mm, no annular, M3")
+    (tags "mounting hole 3.2mm no annular m3")
     (attr virtual)
-    (fp_text reference PAD5 (at 0.254 0.254) (layer F.SilkS)
+    (fp_text reference PAD5 (at -0.254 0) (layer F.SilkS)
       (effects (font (size 1 1) (thickness 0.15)))
     )
@@
       (effects (font (size 1 1) (thickness 0.15)))
     )
-    (pad 1 thru_hole circle (at 0 0) (size 6.4 6.4) (drill 3.2) (layers *.Cu *.Mask)
+    (pad 1 np_thru_hole circle (at 0 0) (size 3.2 3.2) (drill 3.2) (layers *.Cu *.Mask)
       (net 1 /GND))
   )
@@
     (effects (font (size 5 4.2) (thickness 0.8)))
   )
-  (gr_text "POWER\nON" (at 16.256 25.908) (layer F.Cu)
+  (gr_text "POWER\nON" (at 14.732 26.162) (layer F.Cu)
     (effects (font (size 3 3) (thickness 0.75)))
   )
-  (gr_text OFF (at -3.048 45.72) (layer F.Cu)
+  (gr_text OFF (at -4.064 45.72) (layer F.Cu)
     (effects (font (size 5 4.2) (thickness 0.8)))
   )
-  (gr_text LOCK (at 35.56 45.72) (layer F.Cu)
+  (gr_text LOCK (at 33.782 45.72) (layer F.Cu)
     (effects (font (size 5 4.2) (thickness 0.8)))
   )
@@
     (polygon
       (pts
-        (xy -15.24 90.424) (xy 428.244 90.424) (xy 428.244 118.872) (xy -15.24 118.364)
+        (xy 428.244 118.872) (xy -14.986 118.872) (xy -15.24 90.424) (xy 428.244 90.424)
+      )
+    )
+    (polygon
+      (pts
+        (xy 37.084 96.266) (xy 37.084 97.028) (xy 37.846 97.028) (xy 37.846 112.014) (xy 37.338 112.014)
+        (xy 37.338 112.776) (xy 39.37 112.776) (xy 39.37 112.014) (xy 38.862 112.014) (xy 38.862 104.902)
+        (xy 170.18 104.902) (xy 170.18 111.76) (xy 169.418 111.76) (xy 169.418 112.522) (xy 171.704 112.522)
+        (xy 171.704 111.76) (xy 170.942 111.76) (xy 170.942 97.028) (xy 171.704 97.028) (xy 171.704 96.266)
+        (xy 169.418 96.266) (xy 169.418 97.028) (xy 170.18 97.028) (xy 170.18 103.886) (xy 38.862 103.886)
+        (xy 38.862 97.028) (xy 39.624 97.028) (xy 39.624 96.266)
       )
     )
@@
     (polygon
       (pts
-        (xy 424.18 10.287) (xy 424.307 10.287) (xy 424.307 75.438) (xy 423.672 75.438) (xy 423.672 75.444459)
+        (xy 424.18 10.287) (xy 424.307 10.287) (xy 424.307 75.438) (xy 423.926 75.438) (xy 423.672 75.444459)
         (xy -12.457291 76.205371) (xy -12.457291 76.2) (xy -12.573 76.2) (xy -12.573 10.16) (xy 424.18 10.16)
       )
