File: nova1200rev3pcb/nova1200_fptest.kicad_pcb (KiCad board)
At the start: 2 copper layers, 397.5 x 101.6 mm, 174 parts, among them J1 Conn_02x26_Odd_Even, J2 Conn_02x05_Top_Bottom, J3 Conn_02x05_Top_Bottom, J4 Conn_02x01, SW1 SW_SPST, SW10 SW_SPST, SW11 SW_SPST, SW12 SW_SPST, SW13 SW_SPST, SW14 SW_SPST, SW15 SW_SPST, SW16 SW_SPST, SW17 SW_SPDT_MSM, SW18 SW_SPDT_MSM, SW19 SW_SPDT_MSM, SW2 SW_SPST, SW20 SW_SPDT_MSM, SW21 SW_SPDT_MSM, SW22 SW_SPDT_MSM, SW23 SW_SPDT_MSM, SW24 SW_SPDT_MSM, SW25 SW_SPDT_MSM, SW26 SW_SPDT_MSM, SW3 SW_SPST, SW4 SW_SPST, SW5 SW_SPST, SW6 SW_SPST, SW7 SW_SPST, SW8 SW_SPST, SW9 SW_SPST, U1 74LS257, U10 74LS173, U11 74LS173, U12 74LS173, U13 74LS173, U14 74LS173, U15 74LS257, U16 74LS42, U17 74LS42, U18 74LS02, U19 74LS06, U2 74LS257, U20 74LS06, U21 74LS06, U22 74LS173, U3 74LS257, U4 74LS257, U5 74LS173, U6 74LS173, U7 74LS173, U8 74LS173, U9 74LS173

Commit message: Removed bak files
Parts:
- H1: value NA -> MountingHole
- R1, R10, R11, R12, R13, R14, R15, R16, R17, R18, R19, R2, R20, R21, R22, R23, R24, R25, R26, R27, R28, R29, R3, R30, R31, R32, R33, R34, R35, R36, R37, R38, R39, R4, R40, R41, R43, R45, R46, R47, R48, R49, R5, R50, R51, R52, R53, R54, R55, R57, R59, R6, R60, R61, R62, R63, R64, R65, R67, R68, R7, R8, R9: footprint Resistor_THT:R_Axial_DIN0204_L3.6mm_D1.6mm_P5.08mm_Horizontal -> Resistor_THT:R_Axial_DIN0204_L3.6mm_D1.6mm_P7.62mm_Horizontal
- U1, U10, U11, U12, U13, U14, U15, U16, U17, U2, U22, U3, U4, U5, U6, U7, U8, U9: footprint Package_DIP:DIP-16_W10.16mm -> Package_DIP:DIP-16_W7.62mm
- U18, U19, U20, U21: footprint Package_DIP:DIP-14_W10.16mm -> Package_DIP:DIP-14_W7.62mm
- moved C7 14.0 mm to (378.0, 88.6)
- moved R64 12.4 mm to (214.9, 113.3)
- moved R63 12.4 mm to (214.9, 103.1)
- moved R65 12.4 mm to (214.9, 108.2)
- moved R67 10.1 mm to (381.8, 107.2)
- moved R68 10.1 mm to (381.8, 102.1)
- moved R48 7.88 mm to (344.4, 109.5)
- moved R47 7.88 mm to (344.4, 99.3)
- moved R50 7.50 mm to (373.9, 112.3)
- moved R55 7.11 mm to (108.7, 99.1)
- moved R57 7.11 mm to (108.7, 109.2)
- moved R41 6.86 mm to (277.4, 99.1)
- moved R43 6.86 mm to (277.4, 109.2)
- moved R61 6.62 mm to (175.5, 99.6)
- moved R62 6.62 mm to (175.5, 109.7)
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Connections:
- J1 pad 50: /DEFER -> /EXEC
- J1 pad 52: /EXEC -> /DEFER
Routing:
- net /GND: track 0.00 -> 1051.6 mm
Other:
- net class POWER: clearance 0.5 -> 0.3

Commit message: Rev 3 PCB with gnd hand routed rest autorouted
This PCB is close to the original layout, based on overlay of frontpanel photo (in layout). It does not have space for the onboard keypad and LCD. 10 pin connectors for LCD display and keypad are on the right hand side, next to the Arduino USB connector. Fixes compared to the original V2 are:
- use 1 mm holes for J1 and Arduino
- swapped switch and LED for D13 and D14
- control and data switches are larger (miniature)
- lever UP is 1 for data switches
- longer resistor footprints used for easier mounting
- use normal not wide TTL footprints
- exec and defer corrected on J1

Todo: provide enough mounting holes for frontpanel
Routing:
- net /VCC: track 0.00 -> 1183.9 mm, vias 0 -> 2
- net /D2: track 0.00 -> 632.4 mm, vias 0 -> 1
- net /D3: track 0.00 -> 613.4 mm, vias 0 -> 1
- net /D1: track 0.00 -> 608.9 mm, vias 0 -> 2
- net /D0: track 0.00 -> 607.9 mm, vias 0 -> 4
- net /EXEC: track 0.00 -> 504.5 mm, vias 0 -> 1
- net /ND15: track 0.00 -> 454.0 mm, vias 0 -> 4
- net /ION: track 0.00 -> 438.9 mm, vias 0 -> 4
- net /DEFER: track 0.00 -> 434.3 mm, vias 0 -> 4
- net /ND12: track 0.00 -> 416.4 mm, vias 0 -> 3
- net /FETCH: track 0.00 -> 412.5 mm, vias 0 -> 2
- net /ND10: track 0.00 -> 411.7 mm, vias 0 -> 2
- net /RUN: track 0.00 -> 410.6 mm, vias 0 -> 3
- net /ND14: track 0.00 -> 408.6 mm, vias 0 -> 2
- net /ND11: track 0.00 -> 388.2 mm, vias 0 -> 6
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Other:
- board text removed: "Deposit"

Commit message: Added mounting holes (total to 6) to attach front to frontpanel PCB
Also drawn the line through AC0--AC3 pointing to examine and deposit text
Parts:
- added PAD1: MountingHole_Pad, MountingHole:MountingHole_3.2mm_M3_Pad, F.Cu at (242.3, 19.1)
- added PAD1: MountingHole_Pad, MountingHole:MountingHole_3.2mm_M3_Pad, F.Cu at (242.3, 113.0)
- added PAD1: MountingHole_Pad, MountingHole:MountingHole_3.2mm_M3_Pad, F.Cu at (43.2, 19.1)
- moved R40 1.27 mm to (243.3, 108.0)
Routing:
- net /NA12: track 322.9 -> 332.9 mm
- net /ND15: track 454.0 -> 463.8 mm
- net /FETCH: track 412.5 -> 421.0 mm
- net /SEL12: track 179.7 -> 184.5 mm
- net /ND4: track 352.3 -> 357.1 mm
- net /A0': track 347.8 -> 352.6 mm
- net /NA5: track 238.2 -> 243.0 mm
- net /NA11: track 288.5 -> 293.0 mm
- net /ND2: track 234.3 -> 236.4 mm
- net /ION: track 438.9 -> 441.0 mm
- net /ND11: track 388.2 -> 389.4 mm
- net /ND14: track 408.6 -> 409.8 mm
- net Net-(R40-Pad1): track 26.6 -> 27.2 mm
