File: nova1200rev3pcb/nova1200_fptest.kicad_pcb (KiCad board)
At the start: 2 copper layers, 397.5 x 119.4 mm, 211 parts, among them J1 Conn_02x26_Odd_Even, J10 Conn_01x01_Male, J11 Conn_01x04_Female, J12 Conn_01x04_Female, J13 Conn_01x01_Male, J14 Conn_01x01_Male, J15 Conn_01x04_Female, J16 Conn_01x04_Female, J17 Conn_01x04_Female, J18 Conn_01x04_Male, J19 Conn_01x04_Male, J2 Conn_02x05_Odd_Even, J20 Conn_01x01_Male, J24 Conn_01x06_Male, J3 Conn_02x09_Odd Even, J4 Conn_01x02_Male, J5 Conn_01x03_Female, J6 Conn_02x05_Odd_Even, J7 Conn_01x04, J8 Conn_01x04, J9 Conn_01x05_Male, SW1 SW_SPST, SW10 SW_SPST, SW11 SW_SPST, SW12 SW_SPST, SW13 SW_SPST, SW14 SW_SPST, SW15 SW_SPST, SW16 SW_SPST, SW17 SW_SPDT_MSM, SW18 SW_SPDT_MSM, SW19 SW_SPDT_MSM, SW2 SW_SPST, SW20 SW_SPDT_MSM, SW21 SW_SPDT_MSM, SW22 SW_SPDT_MSM, SW23 SW_SPDT_MSM, SW24 SW_SPDT_MSM, SW25 SW_SPDT_MSM, SW26 SW_SPDT_MSM, SW3 SW_SPST, SW4 SW_SPST, SW5 SW_SPST, SW6 SW_SPST, SW7 SW_SPST, SW8 SW_SPST, SW9 SW_SPST, U1 MCP23017_SP, U10 74LS173, U11 74LS173, U12 74LS173, U13 74LS173, U14 74LS173, U15 MCP23017_SP, U16 74LS42, U17 24LC1025, U18 4051, U19 24LC1025, U2 MCP23017_SP, U20 LM7808_TO220, U21 25LCxxx, U22 Teensy3.2, U23 SFH617A-1, U24 7402, U25 SFH617A-1, U3 MCP23017_SP, U4 MCP23017_SP, U5 74LS173, U6 74LS173, U7 24LC1025, U8 24LC1025, U9 74LS173

Commit message: Modified rev3 PCB for Teensy4.1 and Maker Nano RP2040 compatibility
Parts:
- added R64: 2k2, Resistor_THT:R_Axial_DIN0204_L3.6mm_D1.6mm_P7.62mm_Horizontal, F.Cu at (304.7, 111.3)
- added R65: 3k3, Resistor_THT:R_Axial_DIN0204_L3.6mm_D1.6mm_P7.62mm_Horizontal, F.Cu at (304.7, 113.7)
Connections:
- A1 pad 17: Net-(A1-Pad17) -> /SPIVCC
- A1 pad 18: /SPIVCC -> Net-(A1-Pad18)
- A1 pad 5: /LIGHTINT -> Net-(A1-Pad5)
- C13 pad 1: /VCC -> /SPIVCC
- J19 pad 3: /SDA -> /SCK
- J19 pad 4: /SCK -> /SDA
- J6 pad 9: /TA2 -> Net-(J6-Pad9)
- R55 pad 1: /VCC -> /SPIVCC
- R56 pad 1: /VCC -> /SPIVCC
- U17 pad 1: /VCC -> /SPIVCC
- U17 pad 3: /VCC -> /SPIVCC
- U17 pad 8: /VCC -> /SPIVCC
- U19 pad 1: /VCC -> /SPIVCC
- U19 pad 2: /VCC -> /SPIVCC
- U19 pad 3: /VCC -> /SPIVCC
- U19 pad 8: /VCC -> /SPIVCC
- U22 pad 4: /LIGHTINT -> Net-(A1-Pad5)
- U7 pad 3: /VCC -> /SPIVCC
- U7 pad 8: /VCC -> /SPIVCC
- U8 pad 2: /VCC -> /SPIVCC
- U8 pad 3: /VCC -> /SPIVCC
- U8 pad 8: /VCC -> /SPIVCC
Routing:
- net /LIGHTINT: track 172.6 -> 16.2 mm, vias 1 -> 0
- net Net-(A1-Pad5): track 0.00 -> 150.9 mm, vias 0 -> 1
- net /SPIVCC: track 190.5 -> 310.4 mm, vias 2 -> 4
- net /VCC: track 1619.7 -> 1542.5 mm, vias 2 -> 5
- net /TA2: track 109.8 -> 78.0 mm
- net /GND: track 1918.8 -> 1926.2 mm
- net /SDA: track 810.4 -> 817.5 mm
- net /D0: track 489.8 -> 486.4 mm, vias 3 -> 4
- net /SCK: track 830.3 -> 831.4 mm

Commit message: Moved LCD displays to SPIVCC, use 74HCT4051, plot
Parts:
- U18: value 4051 -> 74HCT4051
Connections:
- C19 pad 1: /VCC -> /SPIVCC
- J11 pad 2: /VCC -> /SPIVCC
- J12 pad 2: /VCC -> /SPIVCC
- J15 pad 2: /VCC -> /SPIVCC
- J16 pad 2: /VCC -> /SPIVCC
- J17 pad 2: /VCC -> /SPIVCC
- J18 pad 2: /VCC -> /SPIVCC
- J19 pad 2: /VCC -> /SPIVCC
- R57 pad 1: /VCC -> /SPIVCC
- R58 pad 1: /VCC -> /SPIVCC
- R59 pad 1: /VCC -> /SPIVCC
- R60 pad 1: /VCC -> /SPIVCC
- R61 pad 1: /VCC -> /SPIVCC
Routing:
- net /SPIVCC: track 310.4 -> 793.5 mm, vias 4 -> 10
- net /VCC: track 1542.5 -> 1473.8 mm, vias 5 -> 12
- net /SDA: track 817.5 -> 822.0 mm
- net /SCK: track 831.4 -> 834.7 mm
- net Net-(J2-Pad13): track 267.3 -> 270.1 mm
- net /ION: track 480.9 -> 483.1 mm
- net /EXEC: track 447.5 -> 448.6 mm
- net Net-(J2-Pad10): track 277.4 -> 278.5 mm
- net /FETCH: track 436.2 -> 437.3 mm
- net /CARRY: track 374.1 -> 375.1 mm
- net /SEL7: track 309.2 -> 310.2 mm
- net Net-(J2-Pad12): track 250.1 -> 251.1 mm
- net Net-(D42-Pad2): track 332.2 -> 331.3 mm
