File: nova1200rev3pcb/noname.kicad_pcb_fixed.kicad_pcb (KiCad board)
At the start: 2 copper layers, 397.5 x 119.4 mm, 211 parts, among them J1 Conn_02x26_Odd_Even, J10 Conn_01x01_Male, J11 Conn_01x04_Female, J12 Conn_01x04_Female, J13 Conn_01x01_Male, J14 Conn_01x01_Male, J15 Conn_01x04_Female, J16 Conn_01x04_Female, J17 Conn_01x04_Female, J18 Conn_01x04_Male, J19 Conn_01x04_Male, J2 Conn_02x05_Odd_Even, J20 Conn_01x01_Male, J24 Conn_01x06_Male, J3 Conn_02x09_Odd Even, J4 Conn_01x02_Male, J5 Conn_01x03_Female, J6 Conn_02x05_Odd_Even, J7 Conn_01x04, J8 Conn_01x04, J9 Conn_01x05_Male, SW1 SW_SPST, SW10 SW_SPST, SW11 SW_SPST, SW12 SW_SPST, SW13 SW_SPST, SW14 SW_SPST, SW15 SW_SPST, SW16 SW_SPST, SW17 SW_SPDT_MSM, SW18 SW_SPDT_MSM, SW19 SW_SPDT_MSM, SW2 SW_SPST, SW20 SW_SPDT_MSM, SW21 SW_SPDT_MSM, SW22 SW_SPDT_MSM, SW23 SW_SPDT_MSM, SW24 SW_SPDT_MSM, SW25 SW_SPDT_MSM, SW26 SW_SPDT_MSM, SW3 SW_SPST, SW4 SW_SPST, SW5 SW_SPST, SW6 SW_SPST, SW7 SW_SPST, SW8 SW_SPST, SW9 SW_SPST, U1 MCP23017_SP, U10 74LS173, U11 74LS173, U12 74LS173, U13 74LS173, U14 74LS173, U15 MCP23017_SP, U16 74LS42, U17 24LC1025, U18 4051, U19 24LC1025, U2 MCP23017_SP, U20 LM7808_TO220, U21 25LCxxx, U22 Teensy3.2, U23 SFH617A-1, U24 7402, U25 SFH617A-1, U3 MCP23017_SP, U4 MCP23017_SP, U5 74LS173, U6 74LS173, U7 24LC1025, U8 24LC1025, U9 74LS173

Commit message: Fixes and documentation of issues in rev3 fron panel PCB
Parts:
- removed J8: Conn_01x04, Connector_PinHeader_2.54mm:PinHeader_1x04_P2.54mm_Vertical
- removed R62, R63: 1K, Resistor_THT:R_Axial_DIN0204_L3.6mm_D1.6mm_P7.62mm_Horizontal
- removed U23, U25: SFH617A-1, Package_DIP:DIP-4_W7.62mm
- moved J5 7.11 mm to (378.0, 132.1)
Connections:
- J3 pad 11: Net-(J3-Pad11) -> Net-(D40-Pad2)
- J3 pad 15: Net-(D40-Pad2) -> Net-(J3-Pad15)
- R54 pad 2: Net-(J3-Pad11) -> Net-(J3-Pad15)
- SW24 pad 1: Net-(J3-Pad16) -> Net-(J3-Pad18)
- SW24 pad 3: Net-(J3-Pad4) -> Net-(J3-Pad18)
- U22 pad 2: /SERIALIN -> /LIGHTINT
- U22 pad 3: /SERIALOUT -> /SERIALIN
- U22 pad 4: /LIGHTINT -> /SERIALOUT
Routing:
- net /SERIALIN: track 193.8 -> 87.2 mm, vias 2 -> 0
- net /SERIALOUT: track 148.5 -> 91.3 mm, vias 3 -> 0
- net /SPIVCC: track 190.5 -> 141.5 mm
- net Net-(J8-Pad1): track 39.3 -> 0.00 mm
- net Net-(J8-Pad2): track 36.9 -> 0.00 mm
- net /GND: track 1918.8 -> 1890.2 mm
- net Net-(J8-Pad4): track 26.6 -> 0.00 mm
- net Net-(J8-Pad3): track 23.4 -> 0.00 mm
- net Net-(J3-Pad15): track 0.00 -> 19.7 mm, vias 0 -> 1
- net Net-(J3-Pad11): track 14.4 -> 0.00 mm, vias 1 -> 0
- net Net-(J3-Pad18): track 284.7 -> 294.0 mm, vias 1 -> 0
- net /VCC: track 1619.7 -> 1627.3 mm
- net /D3: track 543.9 -> 551.0 mm
- net Net-(D40-Pad2): track 237.7 -> 243.9 mm
- net /D2: track 536.8 -> 531.1 mm
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Other:
- board text removed: "Cloop"
