File: nova1200rev3pcb/nova1200_fptest_alt.kicad_pcb (KiCad board)
At the start: 2 copper layers, 397.5 x 119.4 mm, 211 parts, among them J1 Conn_02x26_Odd_Even, J10 Conn_01x01_Male, J11 Conn_01x04_Female, J12 Conn_01x04_Female, J13 Conn_01x01_Male, J14 Conn_01x01_Male, J15 Conn_01x04_Female, J16 Conn_01x04_Female, J17 Conn_01x04_Female, J18 Conn_01x04_Male, J19 Conn_01x04_Male, J2 Conn_02x05_Odd_Even, J20 Conn_01x01_Male, J24 Conn_01x06_Male, J3 Conn_02x09_Odd Even, J4 Conn_01x02_Male, J5 Conn_01x03_Female, J6 Conn_02x05_Odd_Even, J7 Conn_01x04, J8 Conn_01x04, J9 Conn_01x05_Male, SW1 SW_SPST, SW10 SW_SPST, SW11 SW_SPST, SW12 SW_SPST, SW13 SW_SPST, SW14 SW_SPST, SW15 SW_SPST, SW16 SW_SPST, SW17 SW_SPDT_MSM, SW18 SW_SPDT_MSM, SW19 SW_SPDT_MSM, SW2 SW_SPST, SW20 SW_SPDT_MSM, SW21 SW_SPDT_MSM, SW22 SW_SPDT_MSM, SW23 SW_SPDT_MSM, SW24 SW_SPDT_MSM, SW25 SW_SPDT_MSM, SW26 SW_SPDT_MSM, SW3 SW_SPST, SW4 SW_SPST, SW5 SW_SPST, SW6 SW_SPST, SW7 SW_SPST, SW8 SW_SPST, SW9 SW_SPST, U1 MCP23017_SP, U10 74LS173, U11 74LS173, U12 74LS173, U13 74LS173, U14 74LS173, U15 MCP23017_SP, U16 74LS42, U17 24LC1025, U18 4051, U19 24LC1025, U2 MCP23017_SP, U20 LM7808_TO220, U21 25LCxxx, U22 Teensy3.2, U23 SFH617A-1, U24 7402, U25 SFH617A-1, U3 MCP23017_SP, U4 MCP23017_SP, U5 74LS173, U6 74LS173, U7 24LC1025, U8 24LC1025, U9 74LS173

Commit message: Fixes and documentation of issues in rev3 fron panel PCB
Parts:
- removed J8: Conn_01x04, Connector_PinHeader_2.54mm:PinHeader_1x04_P2.54mm_Vertical
- removed R62, R63: 1K, Resistor_THT:R_Axial_DIN0204_L3.6mm_D1.6mm_P7.62mm_Horizontal
- removed U23, U25: SFH617A-1, Package_DIP:DIP-4_W7.62mm
- R55, R56: value 1K -> 4K7
- moved J9 37.5 mm to (402.6, 63.8), turned to 90 degrees
- moved J5 34.2 mm to (417.1, 120.1), turned to 0 degrees
- moved C19 13.7 mm to (84.3, 125.0)
- moved R59 9.53 mm to (170.6, 121.9)
- moved R57 9.43 mm to (102.2, 123.7)
- moved R58 9.43 mm to (102.2, 119.5)
- moved C16 7.27 mm to (379.7, 120.1)
- moved U21 6.91 mm to (386.0, 116.3)
- moved J11 6.35 mm to (50.8, 129.5)
- moved J16 6.10 mm to (252.7, 129.5)
- moved C15 6.10 mm to (295.7, 126.0)
- moved R60 6.10 mm to (239.9, 121.9)
- moved U4 6.10 mm to (258.3, 129.3)
- moved R61 5.59 mm to (315.2, 121.9)
- moved J15 5.08 mm to (186.7, 129.5)
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Connections:
- C19 pad 1: /VCC -> Net-(C19-Pad1)
- J24 pad 4: /SSCK -> Net-(J24-Pad4)
- J3 pad 11: Net-(J3-Pad11) -> Net-(D40-Pad2)
- J3 pad 15: Net-(D40-Pad2) -> Net-(J3-Pad15)
- J3 pad 8: Net-(J3-Pad8) -> Net-(D42-Pad1)
- J4 pad 2: Net-(J4-Pad2) -> Net-(C19-Pad1)
- R38 pad 1: Net-(J3-Pad8) -> Net-(R38-Pad1)
- R39 pad 1: Net-(J3-Pad8) -> Net-(R38-Pad1)
- R40 pad 1: Net-(J3-Pad8) -> Net-(R38-Pad1)
- R41 pad 1: Net-(J3-Pad8) -> Net-(R38-Pad1)
- R42 pad 1: Net-(J3-Pad8) -> Net-(R38-Pad1)
- R54 pad 2: Net-(J3-Pad11) -> Net-(J3-Pad15)
- SW24 pad 1: Net-(J3-Pad16) -> Net-(J3-Pad18)
- SW24 pad 3: Net-(J3-Pad4) -> Net-(J3-Pad18)
- U15 pad 8: Net-(J3-Pad8) -> Net-(D42-Pad1)
- U21 pad 6: /SSCK -> Net-(J24-Pad4)
- U22 pad 2: /SERIALIN -> /LIGHTINT
- U22 pad 20: /SSCK -> /SCK
- U22 pad 3: /SERIALOUT -> /SERIALIN
- U22 pad 33: Net-(J4-Pad2) -> Net-(C19-Pad1)
- U22 pad 4: /LIGHTINT -> /SERIALOUT
Routing:
- net /GND: track 1918.8 -> 247.7 mm
- net /VCC: track 1619.7 -> 239.9 mm, vias 2 -> 0
- net /SCK: track 830.3 -> 0.00 mm, vias 5 -> 0
- net /SDA: track 810.4 -> 0.00 mm, vias 2 -> 0
- net /D3: track 543.9 -> 0.00 mm, vias 1 -> 0
- net /D2: track 536.8 -> 0.00 mm, vias 3 -> 0
- net /D1: track 495.5 -> 0.00 mm, vias 2 -> 0
- net /D0: track 489.8 -> 0.00 mm, vias 3 -> 0
- net /ION: track 480.9 -> 0.00 mm, vias 2 -> 0
- net /RUN: track 456.8 -> 0.00 mm, vias 2 -> 0
- net /EXEC: track 447.5 -> 0.00 mm, vias 3 -> 0
- net /NA15: track 440.6 -> 0.00 mm, vias 2 -> 0
- net /FETCH: track 436.2 -> 0.00 mm, vias 3 -> 0
- net /DEFER: track 431.9 -> 0.00 mm, vias 4 -> 0
- net /CONTDATA: track 374.3 -> 0.00 mm, vias 2 -> 0
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Other:
- board text added: "EEPROM3"
- board text removed: "..3"
- board text removed: "Ard n"
- board text removed: "Cloop"
- board text removed: "DWP"
- board text removed: "Kbd"
- board text removed: "Teen"
- board text removed: "WLS"
